Commit message: fix ekf and ros2 control problems

File: jackal/jackal_description/urdf/accessories/camera/D435/_d435.urdf.xacro (robot description, xacro)
@@ -72,5 +72,5 @@
           <origin xyz="${d435_zero_depth_to_glass + d435_glass_to_front} ${-d435_cam_depth_py} 0" rpy="${M_PI/2} 0 ${M_PI/2}"/>
           <geometry>
-            <mesh filename="file://$(find jackal_description)/meshes/d435.dae" />
+            <mesh filename="file://$(find jackal_description)/meshes/d435/d435.dae" />
           </geometry>
           <material name="aluminum"/>

File: jackal/jackal_description/urdf/gz/jackal.gazebo.xacro (robot description, xacro)
@@ -55,5 +55,6 @@
           <update_rate>30</update_rate>
           <visualize>true</visualize>
-          <gz_frame_id>${prefix}camera_depth_optical_frame</gz_frame_id>
+          <gz_frame_id>${prefix}camera_link</gz_frame_id>
+          <!-- if gz_frame_id = ${prefix}camera_depth_optical_frame, rtabmap works -->
           <topic>${prefix}rgbd_camera</topic>
           <camera>
@@ -81,5 +82,5 @@
           <namespace>$(arg namespace)</namespace>
         </ros>
-        <parameters>$(find jackal_description)/config/jackal_control.yaml</parameters>
+        <parameters>$(find jackal_description)/config/ros2_control.yaml</parameters>
         <!-- <controller_manager_name>jackal_controller_manager</controller_manager_name> -->
       </plugin>
